File: PCB/Rev1.2/ergodash.kicad_pcb (KiCad board)
At the start: 2 copper layers, 159.2 x 126.3 mm, 80 parts, among them J1 5PIN, SW1 SW_PUSH, SW10 SW_PUSH, SW11 SW_PUSH, SW12 SW_PUSH, SW13 SW_PUSH, SW14 SW_PUSH, SW15 SW_PUSH, SW16 SW_PUSH, SW17 SW_PUSH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

Commit message: Rev1.0
Parts:
- moved J1 1.83 mm to (197.2, 42.7)
Routing:
- net GND: track 56.5 -> 59.4 mm
- net /sda/uart: track 51.0 -> 52.9 mm
- net /col0: track 324.2 -> 326.2 mm
- net /col1: track 328.9 -> 330.9 mm
